File: SOURCES/KICAD/infinitas.kicad_pcb (KiCad board)
At the start: 2 copper layers, 240 x 70 mm, 210 parts, among them IC101 IC_CS2100CP, IC102 IC_PCA9545APW, IC103 IC_PCA9545APW, IC104 IC_LCMXO2-1200HC-6TG144C, IC105 IC_TLV62565, IC106 IC_ADM811TARTZ, IC107 IC_LM1117MP-5.0, IC108 IC_NCP1117LPST33, IC109 IC_NCP1117LPST33, IC201 IC_XE216-512-TQ128, IC202 IC_NCP4681DSQ25T1G, IC203 IC_IS25LP080D, IC204 IC_NC7WZ07, IC301 IC_ADAU1452, IC302 IC_25AA1024, Q301 Q_STD2805, X101 CON_HDR_02x04, X102 CON_IDC64, X103 CON_IDC64, X104 CON_MicroMatch-10G, X105 CON_MicroFit3_02x02, X201 CON_HDR_02x10, X202 CON_USB_B, X203 CON_HDR_01x04, X301 CON_HDR_02x05

Commit message: Bugfix on Silkscreen
Parts:
- C209, C210, C211, C212, C213, C214, C215, C216, C217, C218, C219, C220, C221, C222, C223, C224, C225, C226, C227, C228, C229, C230, C231, C232, C233: footprint Capacitors_SMD:C_0402 -> rklib:C0402-X7R
- IC101: footprint Housings_SSOP:MSOP-10_3x3mm_Pitch0.5mm -> rklib:MSOP10_3x3mm_Pitch0.5mm
- IC102, IC103: footprint Housings_SSOP:TSSOP-20_4.4x6.5mm_Pitch0.65mm -> rklib:TSSOP20_4.4x6.5mm_Pitch0.65mm
- IC104: footprint Housings_QFP:TQFP-144_20x20mm_Pitch0.5mm -> rklib:TQFP144_20x20mm_Pitch0.5mm
- IC105: footprint TO_SOT_Packages_SMD:SOT-23-5 -> rklib:SOT23-5
- IC106: footprint TO_SOT_Packages_SMD:SOT-143 -> rklib:SOT143
- IC202: footprint TO_SOT_Packages_SMD:SC-70-5 -> rklib:SC70-5
- IC203: footprint Housings_SOIC:SOIC-8_3.9x4.9mm_Pitch1.27mm -> rklib:SOIC8_3.9x4.9mm_Pitch1.27mm
- IC204: footprint TO_SOT_Packages_SMD:SC-70-6 -> rklib:SC70-6
- IC302: footprint Housings_SOIC:SOIJ-8_5.3x5.3mm_Pitch1.27mm -> rklib:SOIJ8_5.3x5.3mm_P1.27mm
- R119, R120, R121, R123, R138, R139, R140, R141, R143, R145, R147, R148, R150, R151, R152, R204: footprint Resistors_SMD:R_Array_Convex_4x0603 -> rklib:RArray_Convex_4x0603
