File: SOURCES/KICAD/infinitas.sch (KiCad schematic (older format))
At the start: 107 parts, among them IC101 PCA9545APW, IC102 CS2100CP, IC103 LCMXO2-1200HC, IC104 TLV62565, IC105 ADM811TARTZ, IC106 LM1117-5.0, IC107 NCP1117LPST33, IC108 NCP1117LPST33, IC109 PCA9545APW, X101 HDR_02x04, X102 IDC_02x32, X103 IDC_02x32, X104 MM-10G, X105 CONN_02X02

Commit message: Add i2c configuration of AK4458
Notice the hack of the i2c modules (LICENSE OF XMOS STUFF IS UNCLEAR)
Other:
- note removed: "TODO:\n- ADC/DAC kopieren"
- moved on the sheet: C101, C133, R101, R102, R103, R104, R105, R106, R107, R108, R109, R110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

Commit message: Bugfix on i2c multiplexer
Parts:
- added R153, R154, R155, R156: RES_47K0_1%_0.125W_Thick_0805, rklib:C0805-RES, symbol RES_4K70_1%_0.125W_Thick_0805
Connections:
- wire segments 617 -> 629
Other:
- note added: "I2C_ADDR: 0xE0"
- note added: "I2C_ADDR: 0xE2"
- note removed: "I2C_MPX1: 0xE0\nI2C_MPX2: 0xE2"
- moved on the sheet: B101, B102, B108, C101, C102, C103, C104, C105, C106, C107, C108, C109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

Commit message: Reset forwarded to FPGA
Connections:
- wire segments 629 -> 630
Changed lines of the file:
@@
 	14550 1150 14550 1950
 Connection ~ 14550 1950
+Text Label 6300 8300 1    39   ~ 0
+~RST
+Wire Wire Line
+	6300 7350 6300 8300
 $EndSCHEMATC

Commit message: Changed USBi connector
Parts:
- removed B108: TEST_1P, rklib:MountingHole_3.2mm_M3_DIN965_Pad, symbol TEST_1P
- removed C122: 22u0, rklib:C0805-X7R, symbol C
- removed IC101, IC109: PCA9545APW, Housings_SSOP:TSSOP-20_4.4x6.5mm_Pitch0.65mm, symbol PCA9545APW
- removed IC102: CS2100CP, Housings_SSOP:MSOP-10_3x3mm_Pitch0.5mm, symbol CS2100CP
- removed IC103: LCMXO2-1200HC, Housings_QFP:TQFP-144_20x20mm_Pitch0.5mm, symbol LCMXO2-1200HC
- removed IC104: TLV62565, TO_SOT_Packages_SMD:SOT-23-5, symbol TLV62565
- removed IC105: ADM811TARTZ, TO_SOT_Packages_SMD:SOT-143, symbol ADM811TARTZ
- removed IC106: LM1117-5.0, TO_SOT_Packages_SMD:SOT-223, symbol LM1117-5.0
- removed IC107, IC108: NCP1117LPST33, TO_SOT_Packages_SMD:SOT-223, symbol LM1117-5.0
- removed L101: 2u20, rklib:MCSDRH73B, symbol L_Small
- removed OSC101: 24MHz576, rklib:ASFL1, symbol 24MHz576
- removed R117, R118, R119, R121, R122, R123, R124, R125, R127, R129, R131, R132, R134, R135, R136: 51R0, Resistors_SMD:R_Array_Convex_4x0603, symbol R_Pack04
- removed R120: 51R0, rklib:C0805-RES, symbol R
- removed R137: 1K00, rklib:C0805-RES, symbol R
- removed R138: 80K6, rklib:C0805-RES, symbol R
- removed R140: 120K, rklib:C0805-RES, symbol R
- removed X101: HDR_02x04, Pin_Headers:Pin_Header_Straight_2x04, symbol Conn_02x04_Odd_Even
- removed X102, X103: IDC_02x32, Connect:IDC_Header_Straight_64pins, symbol Conn_02x32_Odd_Even
- removed X104: MM-10G, rklib:MM-10G, symbol Conn_01x10
- removed X105: CONN_02X02, Connectors_Molex:Connector_Microfit3_Header_02x02_Straight_43045-0428, symbol Conn_02x02_Odd_Even
- added B103: TEST_1P, rklib:MountingHole_3.2mm_M3_DIN965_Pad, symbol TEST_1P
- added C123: CAP_22u0_10V_X5R_0805, rklib:C0805-X7R, symbol CAP_22u0_10V_X5R_0805
- added IC101: IC_CS2100CP, Housings_SSOP:MSOP-10_3x3mm_Pitch0.5mm, symbol IC_CS2100CP
- added IC102, IC103: IC_PCA9545APW, Housings_SSOP:TSSOP-20_4.4x6.5mm_Pitch0.65mm, symbol IC_PCA9545APW
- added IC104: IC_LCMXO2-1200HC-6TG144C, Housings_QFP:TQFP-144_20x20mm_Pitch0.5mm, symbol IC_LCMXO2-1200HC-6TG144C
- added IC105: IC_TLV62565, TO_SOT_Packages_SMD:SOT-23-5, symbol IC_TLV62565
- added IC106: IC_ADM811TARTZ, TO_SOT_Packages_SMD:SOT-143, symbol IC_ADM811TARTZ
- added IC107: IC_LM1117MP-5.0, rklib:SOT223, symbol IC_LM1117MP-5.0
- added IC108, IC109: IC_NCP1117LPST33, rklib:SOT223, symbol IC_NCP1117LPST33
- added L101: IND_2U20_30%_4A5, rklib:MCSDRH73B, symbol IND_2U20_30%_4A5
- added OSC101: OSC_24M576, rklib:ASFL1, symbol OSC_24M576
- added R119, R120, R121, R123, R138, R139, R140, R141, R143, R145, R147, R148, R150, R151, R152: RES_51R0_5%_4x0603, Resistors_SMD:R_Array_Convex_4x0603, symbol RES_51R0_5%_4x0603
- added R122: RES_51R0_1%_0.125W_Thick_0805, rklib:C0805-RES, symbol RES_51R0_1%_0.125W_Thick_0805
- added R153: RES_1K00_1%_0.125W_Thick_0805, rklib:C0805-RES, symbol RES_1K00_1%_0.125W_Thick_0805
- added R154: RES_80K6_1%_0.125W_Thick_0805, rklib:C0805-RES, symbol RES_80K6_1%_0.125W_Thick_0805
- added R156: RES_120K_1%_0.125W_Thick_0805, rklib:C0805-RES, symbol RES_120K_1%_0.125W_Thick_0805
- added X101: CON_HDR_02x04, rklib:HDR_02x04, symbol CON_HDR_02x04
- added X102, X103: CON_IDC64, rklib:IDC64, symbol CON_IDC64
- added X104: CON_MicroMatch-10G, rklib:MM-10G, symbol CON_MicroMatch-10G
- added X105: CON_MicroFit3_02x02, rklib:Microfit3_43045-0428, symbol CON_MicroFit3_02x02
- B101, B102, B104, B105, B106: Value1 (none) -> -; Value2 (none) -> -; digikey (none) -> -
- R101: renamed from R113; digikey ??? -> 311-10.0KCRCT-ND
- R102: renamed from R141; digikey ??? -> 311-2.00KCRCT-ND
- R103: renamed from R142; digikey ??? -> 311-2.00KCRCT-ND
- R104: renamed from R143; digikey ??? -> 311-2.00KCRCT-ND
- R105: renamed from R144; digikey ??? -> 311-2.00KCRCT-ND
- R106: renamed from R145; digikey ??? -> 311-47.0KCRCT-ND
- R107: renamed from R146; digikey ??? -> 311-47.0KCRCT-ND
- R108: renamed from R153; digikey ??? -> 311-47.0KCRCT-ND
- R109: renamed from R154; digikey ??? -> 311-47.0KCRCT-ND
- R110: renamed from R147; digikey ??? -> 311-47.0KCRCT-ND
- R111: renamed from R148; digikey ??? -> 311-47.0KCRCT-ND
- R112: renamed from R149; digikey ??? -> 311-2.00KCRCT-ND
- R113: renamed from R150; digikey ??? -> 311-2.00KCRCT-ND
- R114: renamed from R151; digikey ??? -> 311-2.00KCRCT-ND
- R115: renamed from R152; digikey ??? -> 311-2.00KCRCT-ND
- R116: renamed from R114; digikey ??? -> 311-51.0CRCT-ND
- R117: renamed from R115; digikey ??? -> 311-51.0CRCT-ND
- R124: renamed from R101; digikey ??? -> 311-2.00KCRCT-ND
- R125: renamed from R102; digikey ??? -> 311-2.00KCRCT-ND
- R126: renamed from R103; digikey ??? -> 311-2.00KCRCT-ND
- R127: renamed from R104; digikey ??? -> 311-2.00KCRCT-ND
- R128: renamed from R105; digikey ??? -> 311-47.0KCRCT-ND
- R129: renamed from R106; digikey ??? -> 311-47.0KCRCT-ND
- R130: renamed from R155; digikey ??? -> 311-47.0KCRCT-ND
- R131: renamed from R156; digikey ??? -> 311-47.0KCRCT-ND
- R132: renamed from R107; digikey ??? -> 311-47.0KCRCT-ND
- R133: renamed from R108; digikey ??? -> 311-47.0KCRCT-ND
- R134: renamed from R111; digikey ??? -> 311-2.00KCRCT-ND
- R135: renamed from R112; digikey ??? -> 311-2.00KCRCT-ND
- R136: renamed from R109; digikey ??? -> 311-2.00KCRCT-ND
- R137: renamed from R110; digikey ??? -> 311-2.00KCRCT-ND
- R142: renamed from R126; digikey ??? -> 311-51.0CRCT-ND
- R144: renamed from R128; digikey ??? -> 311-51.0CRCT-ND
- R146: renamed from R130; digikey ??? -> 311-51.0CRCT-ND
- R149: renamed from R133; digikey ??? -> 311-51.0CRCT-ND
- renumbered C133 to C101, C101 to C105, C105 to C106, C106 to C107, C107 to C108, C108 to C109, C109 to C110, C110 to C111, C111 to C112, C112 to C113, C113 to C114, C114 to C115, C115 to C116, C116 to C117, C117 to C118, C118 to C119, C119 to C120, C120 to C121, C121 to C122, C123 to C124, C124 to C125, C125 to C126, C126 to C127, C127 to C128, C128 to C129, C129 to C130, C130 to C131, C131 to C132, C132 to C133, R116 to R118, R139 to R155

Commit message: Upgraded to KiCAD 5
Parts:
- B101, B102, B103, B104, B105, B106: symbol TEST_1P -> infinitas-rescue:TEST_1P
- C101, C103, C104, C105, C106, C107, C108, C109, C110, C111, C112, C113, C114, C115, C116, C117, C118, C119, C120, C121, C124, C126, C129, C132: symbol CAP_100n_50V_X7R_0805 -> rk:CAP_100n_50V_X7R_0805
- C102, C122, C125, C127, C128, C130, C131, C133: symbol CAP_10u0_25V_X5R_0805 -> rk:CAP_10u0_25V_X5R_0805
- C123: symbol CAP_22u0_10V_X5R_0805 -> rk:CAP_22u0_10V_X5R_0805
- IC101: symbol IC_CS2100CP -> rk:IC_CS2100CP
- IC102, IC103: symbol IC_PCA9545APW -> rk:IC_PCA9545APW
- IC104: symbol IC_LCMXO2-1200HC-6TG144C -> rk:IC_LCMXO2-1200HC-6TG144C
- IC105: symbol IC_TLV62565 -> rk:IC_TLV62565
- IC106: symbol IC_ADM811TARTZ -> rk:IC_ADM811TARTZ
- IC107: symbol IC_LM1117MP-5.0 -> rk:IC_LM1117MP-5.0
- IC108, IC109: symbol IC_NCP1117LPST33 -> rk:IC_NCP1117LPST33
- L101: symbol IND_2U20_30%_4A5 -> rk:IND_2U20_30%_4A5
- OSC101: symbol OSC_24M576 -> rk:OSC_24M576
- R101: symbol RES_10K0_1%_0.25W_Thin_0805 -> rk:RES_10K0_1%_0.25W_Thin_0805
- R102, R103, R104, R105, R106, R107, R108, R109, R110, R111, R112, R113, R114, R115, R116, R117, R118, R124, R125, R126, R127, R128, R129, R130, R131, R132, R133, R134, R135, R136, R137, R142, R144, R146, R149: symbol RES_4K70_1%_0.125W_Thick_0805 -> rk:RES_4K70_1%_0.125W_Thick_0805
- R119, R120, R121, R123, R138, R139, R140, R141, R143, R145, R147, R148, R150, R151, R152: symbol RES_51R0_5%_4x0603 -> rk:RES_51R0_5%_4x0603
- R122: symbol RES_51R0_1%_0.125W_Thick_0805 -> rk:RES_51R0_1%_0.125W_Thick_0805
- R153: symbol RES_1K00_1%_0.125W_Thick_0805 -> rk:RES_1K00_1%_0.125W_Thick_0805
- R154: symbol RES_80K6_1%_0.125W_Thick_0805 -> rk:RES_80K6_1%_0.125W_Thick_0805
- R155: symbol RES_100K_1%_0.125W_Thick_0805 -> rk:RES_100K_1%_0.125W_Thick_0805
- R156: symbol RES_120K_1%_0.125W_Thick_0805 -> rk:RES_120K_1%_0.125W_Thick_0805
- X101: symbol CON_HDR_02x04 -> rk:CON_HDR_02x04
- X102, X103: symbol CON_IDC64 -> rk:CON_IDC64
- X104: symbol CON_MicroMatch-10G -> rk:CON_MicroMatch-10G
- X105: symbol CON_MicroFit3_02x02 -> rk:CON_MicroFit3_02x02

Commit message: Bugfix on Silkscreen
Parts:
- IC102, IC103: footprint Housings_SSOP:TSSOP-20_4.4x6.5mm_Pitch0.65mm -> rklib:TSSOP20_4.4x6.5mm_Pitch0.65mm
- IC104: footprint Housings_QFP:TQFP-144_20x20mm_Pitch0.5mm -> rklib:TQFP144_20x20mm_Pitch0.5mm
- IC106: footprint TO_SOT_Packages_SMD:SOT-143 -> rklib:SOT143
Changed lines of the file:
@@
 F 0 "IC106" H 7500 10250 39  0000 L CNN
 F 1 "IC_ADM811TARTZ" H 7700 10100 39  0001 C CNN
-F 2 "TO_SOT_Packages_SMD:SOT-143" H 7650 10000 39  0001 C CNN
+F 2 "rklib:SOT143" H 7650 10000 39  0001 C CNN
 F 3 "" H 7500 10250 39  0000 C CNN
 F 4 "ADM811TARTZ" H 7500 10200 39  0000 L CNN "Value1"
@@
 F 0 "IC102" H 12850 1000 39  0000 L CNN
 F 1 "IC_PCA9545APW" H 13100 800 39  0001 C CNN
-F 2 "Housings_SSOP:TSSOP-20_4.4x6.5mm_Pitch0.65mm" H 13100 750 39  0001 C CNN
+F 2 "rklib:TSSOP20_4.4x6.5mm_Pitch0.65mm" H 13100 750 39  0001 C CNN
 F 3 "" H 13100 1600 60  0001 C CNN
 F 4 "PCA9545APW" H 12850 950 39  0000 L CNN "Value1"
@@
 F 0 "IC103" H 12850 2850 39  0000 L CNN
 F 1 "IC_PCA9545APW" H 13100 2650 39  0001 C CNN
-F 2 "Housings_SSOP:TSSOP-20_4.4x6.5mm_Pitch0.65mm" H 13100 2600 39  0001 C CNN
+F 2 "rklib:TSSOP20_4.4x6.5mm_Pitch0.65mm" H 13100 2600 39  0001 C CNN
 F 3 "" H 13100 3450 60  0001 C CNN
 F 4 "PCA9545APW" H 12850 2800 39  0000 L CNN "Value1"
@@
 F 0 "IC104" H 9400 3000 39  0000 L CNN
 F 1 "IC_LCMXO2-1200HC-6TG144C" H 7500 2750 39  0001 C CNN
-F 2 "Housings_QFP:TQFP-144_20x20mm_Pitch0.5mm" H 7500 2650 39  0001 C CNN
+F 2 "rklib:TQFP144_20x20mm_Pitch0.5mm" H 7500 2650 39  0001 C CNN
 F 3 "" H 6600 4350 60  0000 C CNN
 F 4 "LCMXO2-1200HC-6TG144C" H 9400 2950 39  0000 L CNN "Value1"
