File: SOURCES/KICAD/dsp.sch (KiCad schematic (older format))
At the start: 38 parts, among them IC701 ADAU1452, IC702 25AA1024, Q701 STD2805, X701 HEADER_02X05

Commit message: Bugfix on i2c multiplexer
Connections:
- wire segments 139 -> 141
Other:
- note added: "Do not populate when \ndisconnecting from local i2c bus"
- note added: "Populate with 2K00 when \ndisconnecting from local i2c bus"
- moved on the sheet: R710, R711, R713, R714
Changed lines of the file:
@@
 $Descr A3 16535 11693
 encoding utf-8
-Sheet 7 3
+Sheet 3 3
 Title "DSP"
 Date ""
-Rev ""
-Comp "rk"
+Rev "1.0.0"
+Comp "auverdion"
 Comment1 ""
 Comment2 ""
@@
 Text Label 7100 6350 1    39   ~ 0
 MCLK
-Text Label 8000 6350 1    39   ~ 0
-SDA
-Text Label 8100 6350 1    39   ~ 0
-SCL
 $Comp
 L 25AA1024 IC702
@@
 	7400 6050 7400 6400
 Wire Wire Line
-	8000 6050 8000 6350
-Wire Wire Line
-	8100 6050 8100 6350
+	8000 6050 8000 6750
+Wire Wire Line
+	8100 6050 8100 6650
 Wire Wire Line
 	7600 6050 7600 7350
@@
 $EndComp
 Wire Wire Line
-	5350 7200 5200 7200
-Wire Wire Line
-	5350 7200 5350 7250
-Wire Wire Line
-	5200 7150 5200 7250
-Wire Wire Line
-	5150 7700 5400 7700
-Wire Wire Line
-	5150 7600 5400 7600
+	9700 6250 9550 6250
+Wire Wire Line
+	9700 6250 9700 6300
+Wire Wire Line
+	9550 6200 9550 6300
+Wire Wire Line
+	8000 6750 9750 6750
+Wire Wire Line
+	8100 6650 9750 6650
 $Comp
 L R R711
 U 1 1 5A291447
-P 5350 7400
-F 0 "R711" V 5350 7400 39  0000 C CNN
-F 1 "DNP" V 5425 7400 39  0000 C CNN
-F 2 "rklib:C0805-RES" V 5280 7400 50  0001 C CNN
-F 3 "" H 5350 7400 50  0000 C CNN
-	1    5350 7400
+P 9700 6450
+F 0 "R711" V 9700 6450 39  0000 C CNN
+F 1 "DNP" V 9775 6450 39  0000 C CNN
+F 2 "rklib:C0805-RES" V 9630 6450 50  0001 C CNN
+F 3 "" H 9700 6450 50  0000 C CNN
+	1    9700 6450
 	1    0    0    -1
 $EndComp
@@
 L R R710
 U 1 1 5A29143F
-P 5200 7400
-F 0 "R710" V 5200 7400 39  0000 C CNN
-F 1 "DNP" V 5275 7400 39  0000 C CNN
-F 2 "rklib:C0805-RES" V 5130 7400 50  0001 C CNN
-F 3 "" H 5200 7400 50  0000 C CNN
-	1    5200 7400
-	1    0    0    -1
-$EndComp
-Wire Wire Line
-	4650 7700 4850 7700
-Wire Wire Line
-	4850 7600 4650 7600
-Wire Wire Line
-	6000 7700 6000 7600
-Wire Wire Line
-	5900 7700 6000 7700
-Wire Wire Line
-	5900 7800 6100 7800
-Wire Wire Line
-	5900 7900 6100 7900
-Wire Wire Line
-	5400 8000 5150 8000
-Wire Wire Line
-	5400 7900 5150 7900
-Wire Wire Line
-	5400 7800 5150 7800
+P 9550 6450
+F 0 "R710" V 9550 6450 39  0000 C CNN
+F 1 "DNP" V 9625 6450 39  0000 C CNN
+F 2 "rklib:C0805-RES" V 9480 6450 50  0001 C CNN
+F 3 "" H 9550 6450 50  0000 C CNN
+	1    9550 6450
+	1    0    0    -1
+$EndComp
+Wire Wire Line
+	9050 7350 9050 7150
+Wire Wire Line
+	8950 7150 8950 7350
+Wire Wire Line
+	10350 6750 10350 6650
+Wire Wire Line
+	10250 6750 10350 6750
+Wire Wire Line
+	10250 6850 10450 6850
+Wire Wire Line
+	10250 6950 10450 6950
+Wire Wire Line
+	9750 7050 9500 7050
+Wire Wire Line
+	9750 6950 9500 6950
+Wire Wire Line
+	9750 6850 9500 6850
 $Comp
 L +5VD #PWR0165
 U 1 1 590B625E
-P 6000 7600
-F 0 "#PWR0165" H 6000 7450 50  0001 C CNN
-F 1 "+5VD" H 6000 7740 39  0000 C CNN
-F 2 "" H 6000 7600 50  0000 C CNN
-F 3 "" H 6000 7600 50  0000 C CNN
-	1    6000 7600
-	1    0    0    -1
-$EndComp
-Text Label 6100 7800 2    39   ~ 0
+P 10350 6650
+F 0 "#PWR0165" H 10350 6500 50  0001 C CNN
+F 1 "+5VD" H 10350 6790 39  0000 C CNN
+F 2 "" H 10350 6650 50  0000 C CNN
+F 3 "" H 10350 6650 50  0000 C CNN
+	1    10350 6650
+	1    0    0    -1
+$EndComp
+Text Label 10450 6850 2    39   ~ 0
 ~USBRST
-Text Label 6100 7900 2    39   ~ 0
+Text Label 10450 6950 2    39   ~ 0
 MOSI
-NoConn ~ 5900 7600
-Text Label 5150 8000 0    39   ~ 0
+NoConn ~ 10250 6650
+Text Label 9500 7050 0    39   ~ 0
 ~SS
-Text Label 5150 7900 0    39   ~ 0
+Text Label 9500 6950 0    39   ~ 0
 SCLK
-Text Label 5150 7800 0    39   ~ 0
+Text Label 9500 6850 0    39   ~ 0
 MISO
-Text Label 4700 7600 0    39   ~ 0
+Text Label 8950 7300 1    39   ~ 0
 SCL
-Text Label 4700 7700 0    39   ~ 0
+Text Label 9050 7300 1    39   ~ 0
 SDA
 $Comp
 L GND #PWR0166
 U 1 1 590B6249
-P 5900 8000
-F 0 "#PWR0166" H 5900 7750 50  0001 C CNN
-F 1 "GND" H 5900 7850 39  0000 C CNN
-F 2 "" H 5900 8000 50  0000 C CNN
-F 3 "" H 5900 8000 50  0000 C CNN
-	1    5900 8000
+P 10250 7050
+F 0 "#PWR0166" H 10250 6800 50  0001 C CNN
+F 1 "GND" H 10250 6900 39  0000 C CNN
+F 2 "" H 10250 7050 50  0000 C CNN
+F 3 "" H 10250 7050 50  0000 C CNN
+	1    10250 7050
 	1    0    0    -1
 $EndComp
@@
 L Conn_02x05_Odd_Even X701
 U 1 1 590B6242
-P 5600 7800
-F 0 "X701" H 5600 8100 39  0000 C CNN
-F 1 "HEADER_02X05" V 5600 7800 39  0001 C CNN
-F 2 "Pin_Headers:Pin_Header_Straight_2x05" H 5600 6600 50  0001 C CNN
-F 3 "" H 5600 6600 50  0000 C CNN
-	1    5600 7800
+P 9950 6850
+F 0 "X701" H 9950 7150 39  0000 C CNN
+F 1 "HEADER_02X05" V 9950 6850 39  0001 C CNN
+F 2 "Pin_Headers:Pin_Header_Straight_2x05" H 9950 5650 50  0001 C CNN
+F 3 "" H 9950 5650 50  0000 C CNN
+	1    9950 6850
 	1    0    0    -1
 $EndComp
@@
 	0    1    1    0
 $EndComp
-Text HLabel 4650 7600 0    39   Input ~ 0
+Text HLabel 8950 7350 3    39   Input ~ 0
 SCL
-Text HLabel 4650 7700 0    39   BiDi ~ 0
+Text HLabel 9050 7350 3    39   BiDi ~ 0
 SDA
 Text HLabel 7100 6400 3    39   Input ~ 0
@@
 L +3V3 #PWR0167
 U 1 1 5ACA2F10
-P 5200 7150
-F 0 "#PWR0167" H 5200 7000 50  0001 C CNN
-F 1 "+3V3" H 5200 7290 39  0000 C CNN
-F 2 "" H 5200 7150 50  0000 C CNN
-F 3 "" H 5200 7150 50  0000 C CNN
-	1    5200 7150
-	1    0    0    -1
-$EndComp
-Connection ~ 5200 7200
-Wire Wire Line
-	5200 7550 5200 7700
-Connection ~ 5200 7700
-Wire Wire Line
-	5350 7550 5350 7600
-Connection ~ 5350 7600
-Text HLabel 6100 7800 2    39   Output ~ 0
+P 9550 6200
+F 0 "#PWR0167" H 9550 6050 50  0001 C CNN
+F 1 "+3V3" H 9550 6340 39  0000 C CNN
+F 2 "" H 9550 6200 50  0000 C CNN
+F 3 "" H 9550 6200 50  0000 C CNN
+	1    9550 6200
+	1    0    0    -1
+$EndComp
+Connection ~ 9550 6250
+Wire Wire Line
+	9550 6600 9550 6750
+Connection ~ 9550 6750
+Wire Wire Line
+	9700 6600 9700 6650
+Connection ~ 9700 6650
+Text HLabel 10450 6850 2    39   Output ~ 0
 ~USBRST
 $Comp
 L RES_0R00_1%_0.125W_Thick_0805 R713
 U 1 1 5AD8E75C
-P 5000 7600
-F 0 "R713" H 5000 7600 39  0000 C CNN
-F 1 "RES_0R00_1%_0.125W_Thick_0805" H 5000 7425 39  0001 C CNN
-F 2 "rklib:C0805-RES" H 5000 7375 39  0001 C CNN
-F 3 "" H 5000 7600 50  0000 C CNN
-F 4 "0R00" H 5000 7675 39  0000 C CNN "Value1"
-F 5 "1% 0.125W Thick" H 5000 7475 39  0001 C CNN "Value2"
-F 6 "311-0.0ARCT-ND" H 5000 7300 39  0001 C CNN "digikey"
-	1    5000 7600
-	1    0    0    -1
+P 8950 7000
+F 0 "R713" H 8950 7000 39  0000 C CNN
+F 1 "RES_0R00_1%_0.125W_Thick_0805" H 8950 6825 39  0001 C CNN
+F 2 "rklib:C0805-RES" H 8950 6775 39  0001 C CNN
+F 3 "" H 8950 7000 50  0000 C CNN
+F 4 "0R00" H 8950 7075 39  0000 C CNN "Value1"
+F 5 "1% 0.125W Thick" H 8950 6875 39  0001 C CNN "Value2"
+F 6 "311-0.0ARCT-ND" H 8950 6700 39  0001 C CNN "digikey"
+	1    8950 7000
+	0    -1   -1   0
 $EndComp
 $Comp
 L RES_0R00_1%_0.125W_Thick_0805 R714
 U 1 1 5AD8E82F
-P 5000 7700
-F 0 "R714" H 5000 7700 39  0000 C CNN
-F 1 "RES_0R00_1%_0.125W_Thick_0805" H 5000 7525 39  0001 C CNN
-F 2 "rklib:C0805-RES" H 5000 7475 39  0001 C CNN
-F 3 "" H 5000 7700 50  0000 C CNN
-F 4 "0R00" H 5000 7625 39  0000 C CNN "Value1"
-F 5 "1% 0.125W Thick" H 5000 7575 39  0001 C CNN "Value2"
-F 6 "311-0.0ARCT-ND" H 5000 7400 39  0001 C CNN "digikey"
-	1    5000 7700
-	1    0    0    -1
+P 9050 7000
+F 0 "R714" H 9050 7000 39  0000 C CNN
+F 1 "RES_0R00_1%_0.125W_Thick_0805" H 9050 6825 39  0001 C CNN
+F 2 "rklib:C0805-RES" H 9050 6775 39  0001 C CNN
+F 3 "" H 9050 7000 50  0000 C CNN
+F 4 "0R00" H 9050 6925 39  0000 C CNN "Value1"
+F 5 "1% 0.125W Thick" H 9050 6875 39  0001 C CNN "Value2"
+F 6 "311-0.0ARCT-ND" H 9050 6700 39  0001 C CNN "digikey"
+	1    9050 7000
+	0    -1   -1   0
 $EndComp
 $Comp
@@
 	0    -1   -1   0
 $EndComp
+Wire Wire Line
+	8950 6850 8950 6650
+Connection ~ 8950 6650
+Wire Wire Line
+	9050 6850 9050 6750
+Connection ~ 9050 6750
+Text Notes 9800 6350 0    39   ~ 0
+Populate with 2K00 when \ndisconnecting from local i2c bus
+Text Notes 9100 7300 0    39   ~ 0
+Do not populate when \ndisconnecting from local i2c bus
 $EndSCHEMATC

Commit message: Changed USBi connector
Parts:
- removed C703: 5n60, rklib:C0805-X7R, symbol C
- removed C706: 150p, rklib:C0805-X7R, symbol C
- removed FER701, FER702: 600R./100MHz, rklib:C0805-RES, symbol R
- removed IC701: ADAU1452, rklib:QFP72_10x10_EP_Handsoldering, symbol ADAU1452
- removed IC702: 25AA1024, Housings_SOIC:SOIJ-8_5.3x5.3mm_Pitch1.27mm, symbol 25AA1024
- removed JP701: Jumper, Pin_Headers:Pin_Header_Straight_1x02, symbol Jumper_NC_Small
- removed Q701: STD2805, TO_SOT_Packages_SMD:TO-252-2Lead, symbol Q_PNP_BCE
- removed R701: 1K00, rklib:C0805-RES, symbol R
- removed R702, R703, R704, R705, R706: 51R0, rklib:C0805-RES, symbol R
- removed R707: 4K32, rklib:C0805-RES, symbol R
- removed X701: HEADER_02X05, Pin_Headers:Pin_Header_Straight_2x05, symbol Conn_02x05_Odd_Even
- added C303: CAP_5n60_50V_X7R_0805, rklib:C0805-X7R, symbol CAP_5n60_50V_X7R_0805
- added C306: CAP_150p_50V_C0G_0805, rklib:C0805-X7R, symbol CAP_150p_50V_C0G_0805
- added FER301, FER302: FER_600R_600MA_0805, rklib:C0805-RES, symbol FER_600R_600MA_0805
- added IC301: IC_ADAU1452, rklib:QFP72_10x10_EP_Handsoldering, symbol IC_ADAU1452
- added IC302: IC_25AA1024, Housings_SOIC:SOIJ-8_5.3x5.3mm_Pitch1.27mm, symbol IC_25AA1024
- added JP301: CON_JUMPER, rklib:HDR_01x02, symbol CON_JUMPER
- added Q301: Q_STD2805, TO_SOT_Packages_SMD:TO-252-2Lead, symbol Q_STD2805
- added R301: RES_1K00_1%_0.125W_Thick_0805, rklib:C0805-RES, symbol RES_1K00_1%_0.125W_Thick_0805
- added R302, R303, R304, R305, R306: RES_51R0_1%_0.125W_Thick_0805, rklib:C0805-RES, symbol RES_51R0_1%_0.125W_Thick_0805
- added R307: RES_4K32_1%_0.125W_Thick_0805, rklib:C0805-RES, symbol RES_4K32_1%_0.125W_Thick_0805
- added R315, R316: DNP, rklib:C0805-RES, symbol R
- added R317, R318: RES_0R00_1%_0.125W_Thick_0805, rklib:C0805-RES, symbol RES_0R00_1%_0.125W_Thick_0805
- added X301: CON_HDR_02x05, rklib:HDR_02x05, symbol CON_HDR_02x05
- R308: renamed from R708; digikey ??? -> 311-10.0KCRCT-ND
- R309: renamed from R710; Value1 (none) -> DNP; Value2 (none) -> -; digikey (none) -> -
- R310: renamed from R711; Value1 (none) -> DNP; Value2 (none) -> -; digikey (none) -> -
- R313: renamed from R709; digikey ??? -> 311-10.0KCRCT-ND
- R314: renamed from R712; digikey ??? -> 311-10.0KCRCT-ND
- renumbered C701 to C301, C702 to C302, C704 to C304, C705 to C305, C707 to C307, C708 to C308, C709 to C309, C710 to C310, C711 to C311, C712 to C312, C713 to C313, C714 to C314, C715 to C315, C716 to C316, C717 to C317, R713 to R311, R714 to R312
Connections:
- wire segments 141 -> 153
Other:
- note added: "For SPI control by USBi\n- populate R315, R316 with 0R00\n- do not populate R309, R310, R311, R312, R317, R318\n\nFor I2C control by USBi\n- populate R309, R310 with 2K00\n- populate R317, R318 with 0R00\n- do not populate R311, R312, R315, R316\n\nFor I2C control by XE216\n- populate R311, R312, R317, R318 with 0R00\n- do not populate R309, R310, R315, R316"
- note added: "USBi connector"
- note removed: "Do not populate when \ndisconnecting from local i2c bus"
- note removed: "Populate with 2K00 when \ndisconnecting from local i2c bus"
- moved on the sheet: R309, R310, R311, R312

Commit message: Upgraded to KiCAD 5
Parts:
- C301, C304, C308, C313: symbol CAP_10u0_25V_X5R_0805 -> rk:CAP_10u0_25V_X5R_0805
- C302, C305, C307, C309, C310, C311, C312, C314, C315, C316, C317: symbol CAP_100n_50V_X7R_0805 -> rk:CAP_100n_50V_X7R_0805
- C303: symbol CAP_5n60_50V_X7R_0805 -> rk:CAP_5n60_50V_X7R_0805
- C306: symbol CAP_150p_50V_C0G_0805 -> rk:CAP_150p_50V_C0G_0805
- FER301, FER302: symbol FER_600R_600MA_0805 -> rk:FER_600R_600MA_0805
- IC301: symbol IC_ADAU1452 -> rk:IC_ADAU1452
- IC302: symbol IC_25AA1024 -> rk:IC_25AA1024
- JP301: symbol CON_JUMPER -> rk:CON_JUMPER
- Q301: symbol Q_STD2805 -> rk:Q_STD2805
- R301: symbol RES_1K00_1%_0.125W_Thick_0805 -> rk:RES_1K00_1%_0.125W_Thick_0805
- R302, R303, R304, R305, R306: symbol RES_51R0_1%_0.125W_Thick_0805 -> rk:RES_51R0_1%_0.125W_Thick_0805
- R307: symbol RES_4K32_1%_0.125W_Thick_0805 -> rk:RES_4K32_1%_0.125W_Thick_0805
- R308, R313, R314: symbol RES_10K0_1%_0.25W_Thin_0805 -> rk:RES_10K0_1%_0.25W_Thin_0805
- R309, R310, R315, R316: symbol R -> Device:R
- R311, R312, R317, R318: symbol RES_0R00_1%_0.125W_Thick_0805 -> rk:RES_0R00_1%_0.125W_Thick_0805
- X301: symbol CON_HDR_02x05 -> rk:CON_HDR_02x05

Commit message: Bugfix on Silkscreen
Parts:
- IC302: footprint Housings_SOIC:SOIJ-8_5.3x5.3mm_Pitch1.27mm -> rklib:SOIJ8_5.3x5.3mm_P1.27mm
Changed lines of the file:
@@
 	6550 4000 6500 4000
 Wire Wire Line
-	6500 4000 6500 6100
+	6500 4000 6500 4500
 Wire Wire Line
 	6900 6100 6900 6050
@@
 	9000 5700 8950 5700
 Wire Wire Line
-	9000 6100 9000 3600
+	9000 6100 9000 5700
 Connection ~ 8600 6100
 Wire Wire Line
@@
 	8600 3600 8600 3650
 Wire Wire Line
-	9000 3600 6800 3600
+	9000 3600 8600 3600
 Connection ~ 9000 4000
 Wire Wire Line
@@
 	8500 3650 8500 3550
 Wire Wire Line
-	6450 3550 9050 3550
-Wire Wire Line
-	6450 3450 6450 5700
+	6450 3550 8500 3550
+Wire Wire Line
+	6450 3450 6450 3550
 Wire Wire Line
 	6450 4100 6550 4100
@@
 	7000 3650 7000 3500
 Wire Wire Line
-	5850 3500 9100 3500
-Wire Wire Line
-	9100 3500 9100 6150
+	5850 3500 7000 3500
+Wire Wire Line
+	9100 3500 9100 4100
 Wire Wire Line
 	9100 4100 8950 4100
@@
 	7000 6050 7000 6150
 Wire Wire Line
-	7000 6150 9100 6150
+	7000 6150 8500 6150
 Connection ~ 9100 4100
 Wire Wire Line
@@
 	8400 6200 8400 6050
 Wire Wire Line
-	9200 6150 9200 6250
+	9200 6150 9200 6200
 Connection ~ 9200 6200
 Connection ~ 6500 6100
@@
 	7900 7200 7900 6050
 Wire Wire Line
-	7550 7350 7700 7350
-Wire Wire Line
-	8300 7300 8300 7450
+	7550 7350 7600 7350
+Wire Wire Line
+	8300 7300 8300 7350
 Connection ~ 8300 7350
 Wire Wire Line
@@
 	7200 7550 7250 7550
 Wire Wire Line
-	7200 7300 7200 7550
+	7200 7300 7200 7350
 Wire Wire Line
 	7550 7550 7700 7550
@@
 	8300 7350 8550 7350
 Wire Wire Line
-	5600 4600 6550 4600
+	5600 4600 5650 4600
 Wire Wire Line
 	6550 4700 6150 4700
@@
 Connection ~ 5650 4600
 Wire Wire Line
-	6050 4200 6550 4200
-Wire Wire Line
-	6250 3900 6450 3900
+	6050 4200 6300 4200
+Wire Wire Line
+	6250 3900 6300 3900
 Connection ~ 6300 4200
 Connection ~ 6450 3900
 Connection ~ 6300 3900
 Wire Wire Line
-	5300 5400 6550 5400
-Wire Wire Line
-	5900 6000 6400 6000
+	5300 5400 5600 5400
+Wire Wire Line
+	5900 6000 6200 6000
 Wire Wire Line
 	6400 6000 6400 5500
@@
 Connection ~ 5900 5400
 Wire Wire Line
-	5300 5350 5300 5500
+	5300 5350 5300 5400
 Connection ~ 5600 5400
 Connection ~ 5300 5400
 Wire Wire Line
-	7250 8950 7250 9050
-Wire Wire Line
-	7250 9000 8450 9000
+	7250 8950 7250 9000
+Wire Wire Line
+	7250 9000 7550 9000
 Wire Wire Line
 	7550 9000 7550 9050
@@
 Connection ~ 8150 9000
 Wire Wire Line
-	8750 8950 8750 9050
-Wire Wire Line
-	8750 9000 9950 9000
+	8750 8950 8750 9000
+Wire Wire Line
+	8750 9000 9050 9000
 Wire Wire Line
 	9050 9000 9050 9050
@@
 Connection ~ 9650 9000
 Wire Wire Line
-	5850 3450 5850 3900
+	5850 3450 5850 3500
 Connection ~ 5850 3500
 Wire Wire Line
@@
 	10350 6450 10350 6500
 Wire Wire Line
-	10200 6400 10200 6500
-Wire Wire Line
-	8000 6950 10400 6950
-Wire Wire Line
-	8100 6850 10400 6850
+	10200 6400 10200 6450
+Wire Wire Line
+	8000 6950 9050 6950
+Wire Wire Line
+	8100 6850 8950 6850
 $Comp
 L Device:R R310
@@
 	10900 7150 11100 7150
 Wire Wire Line
-	9600 7250 10400 7250
+	9600 7250 9800 7250
 Wire Wire Line
 	10400 7150 10150 7150
@@
 F 0 "IC302" H 7950 7200 39  0000 L CNN
 F 1 "IC_25AA1024" H 8000 7050 39  0001 C CNN
-F 2 "Housings_SOIC:SOIJ-8_5.3x5.3mm_Pitch1.27mm" H 7950 6950 39  0001 C CNN
+F 2 "rklib:SOIJ8_5.3x5.3mm_P1.27mm" H 7950 6950 39  0001 C CNN
 F 3 "" H 8050 7200 39  0000 C CNN
 F 4 "25AA1024" H 7950 7150 39  0000 L CNN "Value1"
@@
 	11100 7150 11100 7450
 Wire Wire Line
-	11100 7450 9500 7450
+	11100 7450 10000 7450
 Wire Wire Line
 	9500 7450 9500 6750
@@
 	8200 6750 8200 6050
 Wire Wire Line
-	6500 6100 9000 6100
+	6500 6100 6900 6100
 $Comp
 L rk:RES_0R00_1%_0.125W_Thick_0805 R318
@@
 Text Notes 10200 8300 0    39   ~ 0
 For SPI control by USBi\n- populate R315, R316 with 0R00\n- do not populate R309, R310, R311, R312, R317, R318\n\nFor I2C control by USBi\n- populate R309, R310 with 2K00\n- populate R317, R318 with 0R00\n- do not populate R311, R312, R315, R316\n\nFor I2C control by XE216\n- populate R311, R312, R317, R318 with 0R00\n- do not populate R309, R310, R315, R316
+Wire Wire Line
+	6500 5600 6500 6100
+Wire Wire Line
+	6500 4500 6500 5300
+Wire Wire Line
+	6500 5300 6500 5600
+Wire Wire Line
+	6900 6100 7500 6100
+Wire Wire Line
+	7500 6100 8600 6100
+Wire Wire Line
+	8600 6100 9000 6100
+Wire Wire Line
+	9000 5700 9000 4000
+Wire Wire Line
+	9000 4000 9000 3600
+Wire Wire Line
+	8600 3600 6900 3600
+Wire Wire Line
+	6450 4100 6450 5700
+Wire Wire Line
+	8500 3550 9050 3550
+Wire Wire Line
+	6450 3550 6450 3900
+Wire Wire Line
+	9100 4100 9100 6150
+Wire Wire Line
+	8500 6150 9100 6150
+Wire Wire Line
+	7000 3500 9100 3500
+Wire Wire Line
+	9200 6200 9200 6250
+Wire Wire Line
+	8300 7350 8300 7450
+Wire Wire Line
+	7600 7350 7700 7350
+Wire Wire Line
+	7200 7350 7200 7550
+Wire Wire Line
+	5950 4600 6550 4600
+Wire Wire Line
+	5650 4600 5950 4600
+Wire Wire Line
+	6300 4200 6550 4200
+Wire Wire Line
+	6450 3900 6450 4100
+Wire Wire Line
+	6300 3900 6450 3900
+Wire Wire Line
+	6200 5400 6550 5400
+Wire Wire Line
+	6200 6000 6400 6000
+Wire Wire Line
+	5900 5400 6200 5400
+Wire Wire Line
+	5600 5400 5900 5400
+Wire Wire Line
+	5300 5400 5300 5500
+Wire Wire Line
+	7250 9000 7250 9050
+Wire Wire Line
+	7550 9000 7850 9000
+Wire Wire Line
+	7850 9000 8150 9000
+Wire Wire Line
+	8150 9000 8450 9000
+Wire Wire Line
+	8750 9000 8750 9050
+Wire Wire Line
+	9050 9000 9350 9000
+Wire Wire Line
+	9350 9000 9650 9000
+Wire Wire Line
+	9650 9000 9950 9000
+Wire Wire Line
+	5850 3500 5850 3900
+Wire Wire Line
+	6900 3600 6800 3600
+Wire Wire Line
+	10200 6450 10200 6500
+Wire Wire Line
+	10200 6950 10400 6950
+Wire Wire Line
+	10350 6850 10400 6850
+Wire Wire Line
+	8950 6850 9700 6850
+Wire Wire Line
+	9050 6950 9750 6950
+Wire Wire Line
+	9750 6950 10200 6950
+Wire Wire Line
+	9700 6850 10350 6850
+Wire Wire Line
+	9800 7250 10400 7250
+Wire Wire Line
+	10000 7450 9500 7450
 $EndSCHEMATC
