File: SOURCES/KICAD/uac2-if.sch (KiCad schematic (older format))
At the start: 57 parts, among them IC201 IC_XE216-512-TQ128, IC202 IC_NCP4681DSQ25T1G, IC203 IC_IS25LP080D, IC204 IC_NC7WZ07, X201 CON_HDR_02x10, X202 CON_USB_B, X203 CON_HDR_01x04

Commit message: Updated VHDL code
Changed lines of the file:
@@
 	10500 1950 10500 6200
 Wire Wire Line
-	6900 1950 10500 1950
+	6900 1950 9400 1950
 Wire Wire Line
 	6900 1950 6900 2000
@@
 Connection ~ 9400 1950
 Wire Wire Line
-	9450 1600 9550 1600
+	9450 1600 9500 1600
 Wire Wire Line
 	9500 2000 9500 1600
@@
 	7200 2000 7200 1900
 Wire Wire Line
-	6550 1800 6550 5900
+	6550 1800 6550 1900
 Wire Wire Line
 	6550 3350 6650 3350
@@
 	7300 5800 7300 5900
 Wire Wire Line
-	6550 5900 9700 5900
+	6550 5900 7300 5900
 Connection ~ 6550 4650
 Wire Wire Line
@@
 Connection ~ 7800 1900
 Wire Wire Line
-	6550 1900 10550 1900
-Wire Wire Line
-	10550 1900 10550 4650
+	6550 1900 7200 1900
+Wire Wire Line
+	10550 1900 10550 3250
 Connection ~ 9700 1900
 Wire Wire Line
@@
 	8700 2000 8700 1800
 Wire Wire Line
-	8700 1800 8800 1800
+	8700 1800 8750 1800
 Wire Wire Line
 	8800 1800 8800 2000
@@
 	10600 2750 10450 2750
 Wire Wire Line
-	10600 1800 10600 5250
-Wire Wire Line
-	6500 1850 10600 1850
+	10600 1800 10600 1850
+Wire Wire Line
+	6500 1850 9300 1850
 Wire Wire Line
 	9300 1850 9300 2000
@@
 Connection ~ 10600 3650
 Wire Wire Line
-	6500 1850 6500 5950
+	6500 1850 6500 2850
 Wire Wire Line
 	6500 2850 6650 2850
@@
 	7900 5800 7900 5950
 Wire Wire Line
-	6500 5950 8900 5950
+	6500 5950 7900 5950
 Connection ~ 6500 5150
 Wire Wire Line
@@
 $EndComp
 Wire Wire Line
-	5750 10100 5750 10200
-Wire Wire Line
-	5750 10150 8350 10150
+	5750 10100 5750 10150
+Wire Wire Line
+	5750 10150 5950 10150
 Wire Wire Line
 	5950 10150 5950 10200
@@
 Connection ~ 7950 10150
 Wire Wire Line
-	8800 10100 8800 10200
-Wire Wire Line
-	8800 10150 10600 10150
+	8800 10100 8800 10150
+Wire Wire Line
+	8800 10150 9000 10150
 Wire Wire Line
 	9000 10150 9000 10200
@@
 	12600 8450 12550 8450
 Wire Wire Line
-	12600 7650 12600 8500
+	12600 7650 12600 7850
 Wire Wire Line
 	12550 8250 12600 8250
@@
 	7400 2000 7400 1800
 Wire Wire Line
-	7400 1800 7500 1800
+	7400 1800 7450 1800
 Wire Wire Line
 	7500 1800 7500 2000
 Wire Wire Line
-	9800 8000 10200 8000
+	9800 8000 10150 8000
 Connection ~ 7450 1800
 Wire Wire Line
@@
 	6450 3450 6650 3450
 Wire Wire Line
-	5900 4950 6650 4950
+	5900 4950 6350 4950
 Text Label 5900 4950 0    39   ~ 0
 SPI_CS
@@
 $EndComp
 Wire Wire Line
-	5600 8050 5900 8050
+	5600 8050 5650 8050
 Wire Wire Line
 	5650 8050 5650 8100
@@
 	6400 1050 6400 1200
 Wire Wire Line
-	7000 1000 7000 1200
+	7000 1000 7000 1050
 Wire Wire Line
 	7000 1050 6850 1050
@@
 $EndComp
 Wire Wire Line
-	8300 7950 8450 7950
-Wire Wire Line
-	8300 7900 8300 8000
+	8300 7950 8400 7950
+Wire Wire Line
+	8300 7900 8300 7950
 Connection ~ 8300 7950
 Wire Wire Line
 	9150 7950 9300 7950
 Wire Wire Line
-	9300 7900 9300 8000
+	9300 7900 9300 7950
 Connection ~ 9300 7950
 Wire Wire Line
@@
 USBD_P
 Wire Wire Line
-	5050 8050 5300 8050
+	5050 8050 5100 8050
 Wire Wire Line
 	5100 7950 5100 8050
@@
 XSYS_RST_N
 Wire Wire Line
-	10800 8000 11250 8000
+	10800 8000 10900 8000
 Wire Wire Line
 	10900 8000 10900 8200
@@
 XMCLK
 Wire Wire Line
-	3950 8850 3950 8950
+	3950 8850 3950 8900
 Wire Wire Line
 	4050 8550 4050 8900
@@
 SDA
 Wire Wire Line
-	7750 6600 7750 6700
+	7750 6600 7750 6650
 Wire Wire Line
 	7750 6650 7900 6650
@@
 	0    1    1    0
 $EndComp
+Wire Wire Line
+	9400 1950 10500 1950
+Wire Wire Line
+	9500 1600 9550 1600
+Wire Wire Line
+	6550 1900 6550 3350
+Wire Wire Line
+	6550 3350 6550 3850
+Wire Wire Line
+	6550 3850 6550 3950
+Wire Wire Line
+	6550 3950 6550 4650
+Wire Wire Line
+	6550 4650 6550 5900
+Wire Wire Line
+	7300 5900 7800 5900
+Wire Wire Line
+	7800 5900 8600 5900
+Wire Wire Line
+	9300 5900 9700 5900
+Wire Wire Line
+	10550 3950 10550 4650
+Wire Wire Line
+	10550 3850 10550 3950
+Wire Wire Line
+	7200 1900 7800 1900
+Wire Wire Line
+	9600 1900 9700 1900
+Wire Wire Line
+	7800 1900 9600 1900
+Wire Wire Line
+	9700 1900 10550 1900
+Wire Wire Line
+	8600 5900 9300 5900
+Wire Wire Line
+	8750 1800 8800 1800
+Wire Wire Line
+	10600 1850 10600 2750
+Wire Wire Line
+	10600 2750 10600 3650
+Wire Wire Line
+	10600 3650 10600 5250
+Wire Wire Line
+	9300 1850 10600 1850
+Wire Wire Line
+	6500 2850 6500 3650
+Wire Wire Line
+	6500 3650 6500 4150
+Wire Wire Line
+	6500 4150 6500 5150
+Wire Wire Line
+	6500 5150 6500 5950
+Wire Wire Line
+	7900 5950 8100 5950
+Wire Wire Line
+	8100 5950 8900 5950
+Wire Wire Line
+	5750 10150 5750 10200
+Wire Wire Line
+	5950 10150 6150 10150
+Wire Wire Line
+	6150 10150 6350 10150
+Wire Wire Line
+	6350 10150 6550 10150
+Wire Wire Line
+	6550 10150 6750 10150
+Wire Wire Line
+	6750 10150 6950 10150
+Wire Wire Line
+	6950 10150 7150 10150
+Wire Wire Line
+	7150 10150 7350 10150
+Wire Wire Line
+	7350 10150 7550 10150
+Wire Wire Line
+	7550 10150 7750 10150
+Wire Wire Line
+	7750 10150 7950 10150
+Wire Wire Line
+	7950 10150 8150 10150
+Wire Wire Line
+	8800 10150 8800 10200
+Wire Wire Line
+	9000 10150 9200 10150
+Wire Wire Line
+	9200 10150 9400 10150
+Wire Wire Line
+	9400 10150 9600 10150
+Wire Wire Line
+	9600 10150 9800 10150
+Wire Wire Line
+	9800 10150 10000 10150
+Wire Wire Line
+	10000 10150 10200 10150
+Wire Wire Line
+	10200 10150 10400 10150
+Wire Wire Line
+	10400 10150 10600 10150
+Wire Wire Line
+	12600 8450 12600 8500
+Wire Wire Line
+	12600 8250 12600 8450
+Wire Wire Line
+	12600 8050 12600 8250
+Wire Wire Line
+	12600 7850 12600 8050
+Wire Wire Line
+	7450 1800 7500 1800
+Wire Wire Line
+	6350 4950 6650 4950
+Wire Wire Line
+	5650 8050 5900 8050
+Wire Wire Line
+	7000 1050 7000 1200
+Wire Wire Line
+	10550 3250 10550 3850
+Wire Wire Line
+	8150 10150 8350 10150
+Wire Wire Line
+	8300 7950 8300 8000
+Wire Wire Line
+	9300 7950 9300 8000
+Wire Wire Line
+	8400 7950 8450 7950
+Wire Wire Line
+	5100 8050 5300 8050
+Wire Wire Line
+	10900 8000 11000 8000
+Wire Wire Line
+	11000 8000 11250 8000
+Wire Wire Line
+	10150 8000 10200 8000
+Wire Wire Line
+	3950 8900 3950 8950
+Wire Wire Line
+	7750 6650 7750 6700
 $EndSCHEMATC
